File: tests/fixtures/validation_gate/kicad_experiment.kicad_sch (KiCad schematic)
At the start: 100 parts, among them J1 VIN_24V, J11 FAN7 2-pin out, J13 TH1 NTC in, J15 TH3 RTD in, J2 MCU pwr sel (5V/VBUS), J23 FAN2 4-pin out, J27 FAN6 3-pin out, J3 FAN1 4-pin out, J31 FAN8 2-pin out, J33 TH2 NTC in, J35 TH4 RTD in, J43 FAN3 4-pin out, J51 FAN9 2-pin out, J63 FAN4 4-pin out, J7 FAN5 3-pin out, J71 FAN10 2-pin out, Q1 AO3401A (RPP P-FET), Q24 AO3401A (HS PWM), Q25 2N7002 (lvl shift), Q26 AO3400A (LS PWM), Q4 AO3401A (HS PWM), Q46 AO3400A (LS PWM), Q5 2N7002 (lvl shift), Q6 AO3400A (LS PWM), Q66 AO3400A (LS PWM), SW2 FAN1 rail select, SW22 FAN2 rail select, SW26 FAN6 rail select, SW28 FAN8 rail select, SW42 FAN3 rail select, SW48 FAN9 rail select, SW6 FAN5 rail select, SW62 FAN4 rail select, SW68 FAN10 rail select, SW8 FAN7 rail select, U2 TPS54302 (24-12V), U24 MAX31865 (TH4), U3 TPS54302 (24-5V), U4 MAX31865 (TH3), U5 MCP23017 tach exp

Commit message: Guard KiCad 10 fields, fix the validation gate, refresh docs
- Fidelity guard: after every akcli write, check that no body_style /
  in_pos_files / lib_symbols entries were lost and that moved labels
  kept their formatting; restore the file and report otherwise.
- Delete labels by file uuid (akcli's match.at needs exact mils and
  silently matched nothing for off-grid labels); match only for labels
  created earlier in the same run.
- Validation gate: the fixture was an already-cleaned board and the
  gate ran cleanup.py against the real board's path. Re-vendor the
  genuine pre-cleanup board, compare against the stored cleanup.py
  output, run plan with --schematic, and add criterion 1.G.e (KiCad 10
  field fidelity).
- Tests: replace kicad-sch-api round-trip/golden tests with file-level
  fidelity tests; Hypothesis tests run in memory (Flag #5 mask removed);
  NTC recipe re-apply must be byte-identical.
- Embed power:PWR_FLAG in the recipe fixture so it resolves without a
  KiCad install.
- README, ROADMAP, testing doc: describe the akcli backend, mark the
  kicad-sch-api sections obsolete, close flags #2, #3 and #5.

Co-Authored-By: Claude Opus 5.5 <noreply@anthropic.com>
Claude-Session: https://claude.ai/code/session_013Ef38BVtJecwHMYUr1n8yG
Parts:
- C1, C5, C9: footprint Capacitor_SMD:CP_Elec_6.3x7.7 -> (none)
- C10, C11, C12, C13, C14, C2, C3, C31, C32, C33, C4, C6, C7, C8: footprint Capacitor_SMD:C_0603_1608Metric -> (none)
- D1, D23, D3: footprint Diode_SMD:D_SOD-123 -> (none)
- D24, D4, D44, D64: footprint Diode_SMD:D_SMA -> (none)
- F1, F2, F3, F4: footprint Resistor_SMD:R_1812_4532Metric -> (none)
- J1, J11, J13, J15, J31, J35, J51, J71: footprint TerminalBlock_Phoenix:TerminalBlock_Phoenix_MKDS-1,5-2_5.08mm -> (none)
- J2: footprint Connector_PinHeader_2.54mm:PinHeader_1x03_P2.54mm_Vertical -> (none)
- J23, J3, J43, J63: footprint TerminalBlock_Phoenix:TerminalBlock_Phoenix_MKDS-1,5-4_5.08mm -> (none)
- J27, J7: footprint TerminalBlock_Phoenix:TerminalBlock_Phoenix_MKDS-1,5-3_5.08mm -> (none)
- J33: value TH2 NTC in -> TH1 NTC in; footprint TerminalBlock_Phoenix:TerminalBlock_Phoenix_MKDS-1,5-2_5.08mm -> (none)
- L1, L2: footprint Inductor_SMD:L_12x12mm_H8mm -> (none)
- Q1, Q24, Q25, Q26, Q4, Q46, Q5, Q6, Q66: footprint Package_TO_SOT_SMD:SOT-23 -> (none)
- R1, R10, R11, R12, R13, R14, R2, R26, R27, R28, R29, R3, R30, R31, R32, R33, R34, R4, R46, R47, R5, R52, R6, R66, R67, R7, R72, R8, R9: footprint Resistor_SMD:R_0603_1608Metric -> (none)
- SW2, SW22, SW26, SW28, SW42, SW48, SW6, SW62, SW68, SW8: footprint Button_Switch_THT:SW_Slide_1P3T_CK_OS103011MA1QN1 -> (none)
- U2, U3: footprint Package_TO_SOT_SMD:SOT-23-6 -> (none)
- U24, U4: footprint Package_SO:SSOP-20_4.4x6.5mm_P0.65mm -> (none)
- U5: footprint Package_SO:SOIC-28W_7.5x17.9mm_P1.27mm -> (none)
- U_MCU: footprint MCU_Module:RaspberryPi_Pico_SMD_TH -> (none)
Connections:
- net SPI_MISO is gone; now on net FAN6_VPLUS: J33.2 (Pin_2), U24.17 (SDO), U4.17 (SDO), U_MCU.21 (GPIO16)
- net TH3_CS is gone; now on net TH2_NTC: J33.1 (Pin_1), U4.16 (~{CS}), U_MCU.22 (GPIO17)
- net TH4_RTD_MINUS is gone; now on net +24V: J35.2 (Pin_2), U24.11 (RTDIN-), U24.12 (FORCE-), U24.6 (REFIN-)
- net +3V3: no longer U5.18 (~{RESET})
- net FAN10_DRIVE: no longer U_MCU.19 (GPIO14)
- net FAN1_PWM: no longer U_MCU.1 (GPIO0)
- net FAN2_PWM: no longer U_MCU.2 (GPIO1)
- net FAN3_PWM: no longer U_MCU.4 (GPIO2)
- net FAN4_PWM: no longer U_MCU.5 (GPIO3)
- net FAN5_DRIVE: no longer U_MCU.6 (GPIO4)
- net FAN6_DRIVE: no longer U_MCU.7 (GPIO5)
- net FAN6_VPLUS: now also C1.2, C10.2, C11.2, C12.2, C14.2, C2.2, C3.2, C31.2, C32.2, C5.2, C6.2, C7.2, C9.2, J1.2 (Pin_2), J13.2 (Pin_2), J23.3 (Pin_3), J27.2 (Pin_2), J3.3 (Pin_3), J43.3 (Pin_3), J63.3 (Pin_3), J7.2 (Pin_2), Q24.3 (D), Q25.2 (S), Q26.2 (S), Q46.2 (S), Q5.2 (S), Q6.2 (S), Q66.2 (S), R1.2, R10.2, R12.2, R3.2, R30.2, R32.2, R5.2, R52.2, R72.2, U2.1 (GND), U24.13 (GND), U24.18 (DGND), U24.19 (GND), U3.1 (GND), U4.13 (GND), U4.18 (DGND), U4.19 (GND), U5.10 (V_{SS}), U_MCU.13 (GND), U_MCU.18 (GND), U_MCU.23 (GND), U_MCU.28 (GND), U_MCU.3 (GND), U_MCU.33 (AGND), U_MCU.38 (GND), U_MCU.8 (GND)
- net FAN7_DRIVE: no longer U_MCU.9 (GPIO6)
- net FAN8_DRIVE: no longer U_MCU.10 (GPIO7)
- net FAN9_DRIVE: no longer U_MCU.17 (GPIO13)
- net FAN9_PLUS: no longer J51.1 (Pin_1)
- net I2C_SDA: no longer U5.13 (SDA)
- net TH4_CS: no longer U_MCU.20 (GPIO15)
- net VSYS_MCU: no longer U_MCU.39 (VSYS)
- removed net GND: C1.2, C10.2, C11.2, C12.2, C14.2, C2.2, C3.2, C31.2, C32.2, C5.2, C6.2, C7.2, C9.2, J1.2 (Pin_2), J13.2 (Pin_2), J23.3 (Pin_3), J27.2 (Pin_2), J3.3 (Pin_3), J43.3 (Pin_3), J63.3 (Pin_3), J7.2 (Pin_2), Q24.3 (D), Q25.2 (S), Q26.2 (S), Q46.2 (S), Q5.2 (S), Q6.2 (S), Q66.2 (S), R1.2, R10.2, R12.2, R3.2, R30.2, R32.2, R5.2, R52.2, R72.2, U2.1 (GND), U24.13 (GND), U24.18 (DGND), U24.19 (GND), U3.1 (GND), U4.13 (GND), U4.18 (DGND), U4.19 (GND), U5.10 (V_{SS}), U5.15 (A0), U5.16 (A1), U5.17 (A2), U_MCU.13 (GND), U_MCU.18 (GND), U_MCU.23 (GND), U_MCU.28 (GND), U_MCU.3 (GND), U_MCU.33 (AGND), U_MCU.38 (GND), U_MCU.8 (GND)
- no-connect marks 28 -> 20
